File: H1FR20/Design/H1FR20.brd (EAGLE design)
At the start: 34.6 x 30 mm, 22 parts, among them J1 U.FL-R-SMT-1_10_, P1 HEXABIT_17.32_NO_P6_P7_P12, U1 STM32G0B1CEU6N, U2 LORA127X-C1-915, X1 XTALL_CSTCE8M00G52

Commit message: -Correct some documentation issues
Parts:
- U2: value LORA127X-C1-915 -> Lora1276-C1-915
Changed lines of the file:
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@@
 </element>
 <element name="P1" library="hexabitz_connectors" library_urn="urn:adsk.eagle:library:20064578" package="HEXABIT_17.32_NO_P6_P7_P12" package3d_urn="urn:adsk.eagle:package:20064634/2" value="HEXABIT_17.32_NO_P6_P7_P12" x="0" y="15.08125" smashed="yes"/>
-<element name="U2" library="HEXABITZ_ICs" library_urn="urn:adsk.eagle:library:20064554" package="LORA127X-C1" package3d_urn="urn:adsk.eagle:package:42421660/4" value="LORA127X-C1-915" x="0.15875" y="17.62125" smashed="yes" rot="R180">
+<element name="U2" library="HEXABITZ_ICs" library_urn="urn:adsk.eagle:library:20064554" package="LORA127X-C1" package3d_urn="urn:adsk.eagle:package:42421660/4" value="Lora1276-C1-915" x="0.15875" y="17.62125" smashed="yes" rot="R180">
 <attribute name="AVAILABILITY" value="Not in stock" x="0.15875" y="17.62125" size="1.778" layer="27" rot="R180" display="off"/>
 <attribute name="CHECK_PRICES" value="https://www.snapeda.com/parts/ESP8266-12E/ESP-12E/AI-Thinker/view-part/?ref=eda" x="0.15875" y="17.62125" size="1.778" layer="27" rot="R180" display="off"/>
