File: H1FR20/Design/H1FR20.sch (EAGLE design)
At the start: 22 parts, among them J1 U.FL-R-SMT-1_10_, P1 HEXABIT_17.32_NO_P6_P7_P12, U1 STM32G0B1CEU6N, U2 LORA127X-C1-915, X1 XTALL_CSTCE8M00G52

Commit message: -Correct some documentation issues
Parts:
- U2: value LORA127X-C1-915 -> Lora1276-C1-915
Changed lines of the file:
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@@
 <part name="SWD" library="HEXABITZ_CONNECTION_PARTS" library_urn="urn:adsk.eagle:library:20064553" deviceset="PINHD-1X3" device="SWD" package3d_urn="urn:adsk.eagle:package:42172676/2"/>
 <part name="P1" library="hexabitz_connectors" library_urn="urn:adsk.eagle:library:20064578" deviceset="HEXABIT_?_NO_P6_P7_P12" device="17.32" package3d_urn="urn:adsk.eagle:package:20064634/2"/>
-<part name="U2" library="HEXABITZ_ICs" library_urn="urn:adsk.eagle:library:20064554" deviceset="LORA127X-C1" device="" package3d_urn="urn:adsk.eagle:package:42421660/4" value="LORA127X-C1-915"/>
+<part name="U2" library="HEXABITZ_ICs" library_urn="urn:adsk.eagle:library:20064554" deviceset="LORA127X-C1" device="" package3d_urn="urn:adsk.eagle:package:42421660/4" value="Lora1276-C1-915"/>
 <part name="J1" library="HEXABITZ_CONNECTION_PARTS" library_urn="urn:adsk.eagle:library:20064553" deviceset="U.FL-R-SMT-1_10_" device="" package3d_urn="urn:adsk.eagle:package:42403633/2"/>
 <part name="GND3" library="supply1" library_urn="urn:adsk.eagle:library:371" deviceset="GND" device=""/>
